File: amp_control_board.kicad_pcb (KiCad board)
At the start: 2 copper layers, 100.1 x 61 mm, 90 parts, among them J1 Conn_01x03_Male, J2 Conn_01x04_Female, J3 Conn_01x03_Male, J4 Screw_Terminal_01x02, J5 Conn_01x04_Female, J6 Conn_02x03_Odd_Even, J7 Conn_01x03_Male, J8 USB_B_Mini, M1 Fan_4pin, M2 Fan_4pin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

Commit message: small cleanup
Parts:
- added DS1: HY1602E, Display:WC1602A, F.Cu at (134.6, 29.2)
Routing:
- net Net-(DS1-Pad7): vias 0 -> 1
- net Net-(DS1-Pad15): vias 0 -> 1
- net GND: vias 140 -> 138
Changed lines of the file:
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@@
     (tracks 907)
     (zones 0)
-    (modules 90)
-    (nets 68)
+    (modules 91)
+    (nets 84)
   )
   (page A4)
@@
   (net 66 USB_M)
   (net 67 USB_DT)
+  (net 68 "Net-(DS1-Pad15)")
+  (net 69 "Net-(DS1-Pad7)")
+  (net 70 "Net-(DS1-Pad16)")
+  (net 71 "Net-(DS1-Pad14)")
+  (net 72 "Net-(DS1-Pad13)")
+  (net 73 "Net-(DS1-Pad12)")
+  (net 74 "Net-(DS1-Pad11)")
+  (net 75 "Net-(DS1-Pad10)")
+  (net 76 "Net-(DS1-Pad9)")
+  (net 77 "Net-(DS1-Pad8)")
+  (net 78 "Net-(DS1-Pad6)")
+  (net 79 "Net-(DS1-Pad5)")
+  (net 80 "Net-(DS1-Pad4)")
+  (net 81 "Net-(DS1-Pad3)")
+  (net 82 "Net-(DS1-Pad2)")
+  (net 83 "Net-(DS1-Pad1)")
   (net_class Default "This is the default net class."
     (clearance 0.2)
@@
     (add_net "Net-(D2-Pad2)")
     (add_net "Net-(D3-Pad1)")
+    (add_net "Net-(DS1-Pad1)")
+    (add_net "Net-(DS1-Pad10)")
+    (add_net "Net-(DS1-Pad11)")
+    (add_net "Net-(DS1-Pad12)")
+    (add_net "Net-(DS1-Pad13)")
+    (add_net "Net-(DS1-Pad14)")
+    (add_net "Net-(DS1-Pad15)")
+    (add_net "Net-(DS1-Pad16)")
+    (add_net "Net-(DS1-Pad2)")
+    (add_net "Net-(DS1-Pad3)")
+    (add_net "Net-(DS1-Pad4)")
+    (add_net "Net-(DS1-Pad5)")
+    (add_net "Net-(DS1-Pad6)")
+    (add_net "Net-(DS1-Pad7)")
+    (add_net "Net-(DS1-Pad8)")
+    (add_net "Net-(DS1-Pad9)")
     (add_net "Net-(J6-Pad3)")
     (add_net "Net-(J6-Pad4)")
@@
     (add_net VIN_DC)
   )
+  (module Display:WC1602A (layer F.Cu)
+    (at 134.62 29.21)
+    (descr "LCD 16x2 http://www.wincomlcd.com/pdf/WC1602A-SFYLYHTC06.pdf")
+    (tags "LCD 16x2 Alphanumeric 16pin")
+    (fp_text reference DS1 (at -5.82 -3.81) (layer F.SilkS)
+      (effects (font (size 1 1) (thickness 0.15)))
+    )
+    (fp_text value HY1602E (at -4.31 34.66) (layer F.Fab)
+      (effects (font (size 1 1) (thickness 0.15)))
+    )
+    (fp_arc (start 0.20066 8.49884) (end -0.29972 8.49884) (angle 90) (layer F.SilkS) (width 0.12))
+    (fp_arc (start 0.20066 22.49932) (end 0.20066 22.9997) (angle 90) (layer F.SilkS) (width 0.12))
+    (fp_arc (start 63.70066 22.49932) (end 64.20104 22.49932) (angle 90) (layer F.SilkS) (width 0.12))
+    (fp_arc (start 63.7 8.5) (end 63.7 8) (angle 90) (layer F.SilkS) (width 0.12))
+    (fp_text user %R (at 30.37 14.74) (layer F.Fab)
+      (effects (font (size 1 1) (thickness 0.1)))
+    )
+    (fp_line (start -8.14 33.64) (end 72.14 33.64) (layer F.SilkS) (width 0.12))
+    (fp_line (start 72.14 33.64) (end 72.14 -2.64) (layer F.SilkS) (width 0.12))
+    (fp_line (start 72.14 -2.64) (end -7.34 -2.64) (layer F.SilkS) (width 0.12))
+    (fp_line (start -8.14 -2.64) (end -8.14 33.64) (layer F.SilkS) (width 0.12))
+    (fp_line (start -8.13 -2.64) (end -7.34 -2.64) (layer F.SilkS) (width 0.12))
+    (fp_line (start -8.25 -2.75) (end -8.25 33.75) (layer F.CrtYd) (width 0.05))
+    (fp_line (start -8.25 33.75) (end 72.25 33.75) (layer F.CrtYd) (width 0.05))
+    (fp_line (start 72.25 -2.75) (end 72.25 33.75) (layer F.CrtYd) (width 0.05))
+    (fp_line (start -1.5 -3) (end 1.5 -3) (layer F.SilkS) (width 0.12))
+    (fp_line (start -8.25 -2.75) (end 72.25 -2.75) (layer F.CrtYd) (width 0.05))
+    (fp_line (start 1 -2.5) (end 0 -1.5) (layer F.Fab) (width 0.1))
+    (fp_line (start 0 -1.5) (end -1 -2.5) (layer F.Fab) (width 0.1))
+    (fp_line (start -1 -2.5) (end -8 -2.5) (layer F.Fab) (width 0.1))
+    (fp_line (start 0.2 8) (end 63.7 8) (layer F.SilkS) (width 0.12))
+    (fp_line (start -0.29972 22.49932) (end -0.29972 8.5) (layer F.SilkS) (width 0.12))
+    (fp_line (start 63.70066 23) (end 0.2 23) (layer F.SilkS) (width 0.12))
+    (fp_line (start 64.2 8.5) (end 64.2 22.5) (layer F.SilkS) (width 0.12))
+    (fp_line (start -5 3) (end 68 3) (layer F.SilkS) (width 0.12))
+    (fp_line (start 68 3) (end 68 28) (layer F.SilkS) (width 0.12))
+    (fp_line (start 68 28) (end -5 28) (layer F.SilkS) (width 0.12))
+    (fp_line (start -5 28) (end -5 3) (layer F.SilkS) (width 0.12))
+    (fp_line (start 1 -2.5) (end 72 -2.5) (layer F.Fab) (width 0.1))
+    (fp_line (start 72 -2.5) (end 72 33.5) (layer F.Fab) (width 0.1))
+    (fp_line (start 72 33.5) (end -8 33.5) (layer F.Fab) (width 0.1))
+    (fp_line (start -8 33.5) (end -8 -2.5) (layer F.Fab) (width 0.1))
+    (pad "" thru_hole circle (at 69.5 0) (size 3 3) (drill 2.5) (layers *.Cu *.Mask))
+    (pad "" thru_hole circle (at 69.49948 31.0007) (size 3 3) (drill 2.5) (layers *.Cu *.Mask))
+    (pad "" thru_hole circle (at -5.4991 31.0007) (size 3 3) (drill 2.5) (layers *.Cu *.Mask))
+    (pad "" thru_hole circle (at -5.4991 0) (size 3 3) (drill 2.5) (layers *.Cu *.Mask))
+    (pad 16 thru_hole oval (at 38.1 0) (size 1.8 2.6) (drill 1.2) (layers *.Cu *.Mask)
+      (net 70 "Net-(DS1-Pad16)"))
+    (pad 15 thru_hole oval (at 35.56 0) (size 1.8 2.6) (drill 1.2) (layers *.Cu *.Mask)
+      (net 68 "Net-(DS1-Pad15)"))
+    (pad 14 thru_hole oval (at 33.02 0) (size 1.8 2.6) (drill 1.2) (layers *.Cu *.Mask)
+      (net 71 "Net-(DS1-Pad14)"))
+    (pad 13 thru_hole oval (at 30.48 0) (size 1.8 2.6) (drill 1.2) (layers *.Cu *.Mask)
+      (net 72 "Net-(DS1-Pad13)"))
+    (pad 12 thru_hole oval (at 27.94 0) (size 1.8 2.6) (drill 1.2) (layers *.Cu *.Mask)
+      (net 73 "Net-(DS1-Pad12)"))
+    (pad 11 thru_hole oval (at 25.4 0) (size 1.8 2.6) (drill 1.2) (layers *.Cu *.Mask)
+      (net 74 "Net-(DS1-Pad11)"))
+    (pad 10 thru_hole oval (at 22.86 0) (size 1.8 2.6) (drill 1.2) (layers *.Cu *.Mask)
+      (net 75 "Net-(DS1-Pad10)"))
+    (pad 9 thru_hole oval (at 20.32 0) (size 1.8 2.6) (drill 1.2) (layers *.Cu *.Mask)
+      (net 76 "Net-(DS1-Pad9)"))
+    (pad 8 thru_hole oval (at 17.78 0) (size 1.8 2.6) (drill 1.2) (layers *.Cu *.Mask)
+      (net 77 "Net-(DS1-Pad8)"))
+    (pad 7 thru_hole oval (at 15.24 0) (size 1.8 2.6) (drill 1.2) (layers *.Cu *.Mask)
+      (net 69 "Net-(DS1-Pad7)"))
+    (pad 6 thru_hole oval (at 12.7 0) (size 1.8 2.6) (drill 1.2) (layers *.Cu *.Mask)
+      (net 78 "Net-(DS1-Pad6)"))
+    (pad 5 thru_hole oval (at 10.16 0) (size 1.8 2.6) (drill 1.2) (layers *.Cu *.Mask)
+      (net 79 "Net-(DS1-Pad5)"))
+    (pad 4 thru_hole oval (at 7.62 0) (size 1.8 2.6) (drill 1.2) (layers *.Cu *.Mask)
+      (net 80 "Net-(DS1-Pad4)"))
+    (pad 3 thru_hole oval (at 5.08 0) (size 1.8 2.6) (drill 1.2) (layers *.Cu *.Mask)
+      (net 81 "Net-(DS1-Pad3)"))
+    (pad 2 thru_hole oval (at 2.54 0) (size 1.8 2.6) (drill 1.2) (layers *.Cu *.Mask)
+      (net 82 "Net-(DS1-Pad2)"))
+    (pad 1 thru_hole rect (at 0 0) (size 1.8 2.6) (drill 1.2) (layers *.Cu *.Mask)
+      (net 83 "Net-(DS1-Pad1)"))
+    (model ${KISYS3DMOD}/Display.3dshapes/WC1602A.wrl
+      (at (xyz 0 0 0))
+      (scale (xyz 1 1 1))
+      (rotate (xyz 0 0 0))
+    )
+  )
   (module graphics_own:sound_7x7mm (layer F.Cu)
     (at 179.07 93.98)
@@
   (segment (start 162.088 120.36) (end 161.9625 120.4855) (width 0.25) (layer F.Cu) (net 2))
   (via (at 161.29 88.9) (size 0.8) (drill 0.4) (layers F.Cu B.Cu) (net 2))
-  (via (at 151.13 69.85) (size 0.8) (drill 0.4) (layers F.Cu B.Cu) (net 2))
   (via (at 154.94 69.85) (size 0.8) (drill 0.4) (layers F.Cu B.Cu) (net 2))
   (via (at 152.4 72.39) (size 0.8) (drill 0.4) (layers F.Cu B.Cu) (net 2))
@@
   (via (at 163.83 83.82) (size 0.8) (drill 0.4) (layers F.Cu B.Cu) (net 2))
   (via (at 166.37 83.82) (size 0.8) (drill 0.4) (layers F.Cu B.Cu) (net 2))
-  (via (at 171.45 71.12) (size 0.8) (drill 0.4) (layers F.Cu B.Cu) (net 2))
   (via (at 160.02 72.39) (size 0.8) (drill 0.4) (layers F.Cu B.Cu) (net 2))
   (via (at 196.85 81.28) (size 0.8) (drill 0.4) (layers F.Cu B.Cu) (net 2))
@@
   (segment (start 169.92459 125.222) (end 211.328 125.222) (width 0.25) (layer F.Cu) (net 67))
   (segment (start 169.16 124.45741) (end 169.92459 125.222) (width 0.25) (layer F.Cu) (net 67))
+  (via (at 171.45 71.12) (size 0.8) (drill 0.4) (layers F.Cu B.Cu) (net 68))
+  (via (at 151.13 69.85) (size 0.8) (drill 0.4) (layers F.Cu B.Cu) (net 69))
   (zone (net 0) (net_name "") (layer F.Cu) (hatch edge 0.508)
     (connect_pads (clearance 0.508))
